File: DeskPCB/DeskPCB.sch (KiCad schematic (older format))
At the start: 14 parts, among them J1 8P8C, J2 8P8C, J3 USB_B_Micro, J4 Conn_01x05_Female, J5 USB_B_Micro, U1 74125, U2 WeMos_D1_mini

Commit message: updates fixes
Parts:
- J3, J5: symbol Connector:USB_B_Micro -> DeskPCB:USB_B_Micro
Connections:
- no-connect marks 26 -> 27
Changed lines of the file:
@@
 EESchema Schematic File Version 4
-LIBS:DeskPCB-cache
 EELAYER 30 0
 EELAYER END
@@
 $EndComp
 $Comp
-L Connector:USB_B_Micro J5
+L DeskPCB:USB_B_Micro J5
 U 1 1 5DEA3BDD
 P 8100 3800
@@
 $EndComp
 $Comp
-L Connector:USB_B_Micro J3
+L DeskPCB:USB_B_Micro J3
 U 1 1 5DEAE556
 P 8050 5050
@@
 	1    0    0    -1
 $EndComp
+NoConn ~ 4400 5400
 $EndSCHEMATC
