File: TheListener/Mothership/Mothership.kicad_pcb (KiCad board)
At the start: 2 copper layers, 81 parts, among them J1 RJ45, J2 RJ45, J3 RJ45, J4 RJ45, J5 RJ45, J6 RJ45, J7 RJ45, J8 RJ45, J9 Conn_01x02_Female, U1 SP3491, U10 AMS1117-3.3, U11 NID35-5, U12 Teensy3.5, U2 SP3491, U3 SP3491, U4 SP3491, U5 SP3491, U6 SP3491, U7 SP3491, U8 SP3491, U9 AMS1117-3.3

Commit message: wip
Parts:
- moved R28 2.24 mm to (73.5, 89.0), turned to 180 degrees
- moved R31 1.80 mm to (94.2, 89.0), turned to 180 degrees
- moved R29 1.60 mm to (79.5, 89.0), turned to 180 degrees
- moved R32 1.60 mm to (89.8, 89.0), turned to 0 degrees
- moved R19 1.41 mm to (99.2, 69.5), turned to 0 degrees
- moved R22 0.90 mm to (91.5, 69.5), turned to 0 degrees
- moved R26 0.75 mm to (78.0, 68.5)
- moved R17 0.56 mm to (103.5, 74.5)
- moved R18 0.56 mm to (101.0, 74.5)
- moved R23 0.35 mm to (88.2, 68.5)
- moved R24 0.35 mm to (85.8, 74.5)
- moved R21 0.25 mm to (93.2, 74.5)
- moved R27 0.25 mm to (73.0, 74.5)
- moved R30 0.25 mm to (83.0, 84.0)
Routing:
- net R_5: track 14.3 -> 48.2 mm
- net T_6: track 14.3 -> 42.0 mm
- net T_5: track 14.3 -> 36.6 mm
- net R_8: track 14.3 -> 35.7 mm
- net Net-(R17-Pad1): track 21.0 -> 2.00 mm
- net Net-(R24-Pad1): track 19.4 -> 1.97 mm
- net Net-(R27-Pad1): track 18.8 -> 2.02 mm
- net R_7: track 14.3 -> 29.6 mm
- net R_1: track 14.3 -> 27.0 mm
- net Net-(R30-Pad1): track 12.4 -> 1.81 mm
- net Net-(R20-Pad1): track 12.2 -> 1.88 mm
- net T_1: track 14.3 -> 22.6 mm
- net T_8: track 14.3 -> 22.3 mm
- net R_6: track 10.8 -> 18.4 mm, vias 1 -> 2
- net Net-(R18-Pad1): track 6.95 -> 1.71 mm
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
Commit message: wip
Parts:
- moved R23 1.41 mm to (87.2, 69.5), turned to 180 degrees
- moved R26 1.41 mm to (77.0, 69.5), turned to 180 degrees
- moved R25 1.06 mm to (82.2, 69.5), turned to 180 degrees
Routing:
- net R_3: track 14.3 -> 49.3 mm
- net R_4: track 14.3 -> 42.1 mm
- net T_4: track 14.3 -> 40.3 mm
- net R_2: track 14.3 -> 29.2 mm
- net T_3: track 14.3 -> 28.6 mm
- added copper zone on B.Cu, net (none)

Commit message: updates
Routing:
- net VCC2: track 205.3 -> 211.7 mm, vias 33 -> 30
- net VCC1: track 226.0 -> 232.2 mm, vias 33 -> 30
- added copper zone on B.Cu, net GND
- removed copper zone on B.Cu, net (none)
Changed lines of the file:
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@@
     (thickness 1.6)
     (drawings 0)
-    (tracks 749)
+    (tracks 745)
     (zones 0)
     (modules 81)
@@
     (user_trace_width 5)
     (trace_clearance 0.25)
-    (zone_clearance 0.5)
-    (zone_45_only no)
+    (zone_clearance 2)
+    (zone_45_only yes)
     (trace_min 0.2)
     (via_size 0.8)
@@
   (segment (start 75.5 94.75) (end 75.5 94.75) (width 0.25) (layer F.Cu) (net 43) (status 40000))
   (via (at 75.5 94.75) (size 0.8) (drill 0.4) (layers F.Cu B.Cu) (net 43) (status 40000))
+  (via (at 75.5 91.25) (size 0.8) (drill 0.4) (layers F.Cu B.Cu) (net 43) (status 40000))
+  (segment (start 75.5 94.75) (end 75.5 91.25) (width 0.25) (layer B.Cu) (net 43))
+  (segment (start 75.5 91.25) (end 76.5 91.25) (width 0.25) (layer F.Cu) (net 43))
+  (segment (start 76.5 91.25) (end 78.75 89) (width 0.25) (layer F.Cu) (net 43))
   (segment (start 85.25 101) (end 85.25 94.75) (width 0.25) (layer F.Cu) (net 44) (status 40000))
   (segment (start 86.98 102.75) (end 86.98 102.73) (width 0.25) (layer F.Cu) (net 44) (status 40000))
@@
   (via (at 127.3 35.9) (size 0.8) (drill 0.4) (layers F.Cu B.Cu) (net 68) (status 40000))
   (via (at 123.3 27.9) (size 0.8) (drill 0.4) (layers F.Cu B.Cu) (net 68) (status 40000))
-  (via (at 125.3 35.9) (size 0.8) (drill 0.4) (layers F.Cu B.Cu) (net 68) (status 40000))
   (via (at 121.3 27.9) (size 0.8) (drill 0.4) (layers F.Cu B.Cu) (net 68) (status 40000))
-  (via (at 123.3 35.9) (size 0.8) (drill 0.4) (layers F.Cu B.Cu) (net 68) (status 40000))
-  (via (at 121.3 35.9) (size 0.8) (drill 0.4) (layers F.Cu B.Cu) (net 68) (status 40000))
   (via (at 127.3 29.9) (size 0.8) (drill 0.4) (layers F.Cu B.Cu) (net 68) (status 40000))
   (via (at 123.3 33.9) (size 0.8) (drill 0.4) (layers F.Cu B.Cu) (net 68) (status 40000))
@@
   (segment (start 116.75 46) (end 116.75 62) (width 2) (layer F.Cu) (net 68) (status 40000))
   (segment (start 116.75 35.75) (end 116.75 46) (width 2) (layer F.Cu) (net 68) (status 40000))
+  (segment (start 123.3 42.05) (end 123.3 35.8) (width 0.25) (layer F.Cu) (net 68))
   (segment (start 116.75 96.5) (end 113.5 93) (width 2) (layer F.Cu) (net 69) (status 40000))
   (segment (start 77.25 93) (end 60.25 93) (width 2) (layer F.Cu) (net 69) (status 40000))
@@
   (via (at 121.5 126.5) (size 0.8) (drill 0.4) (layers F.Cu B.Cu) (net 69) (status 40000))
   (via (at 121.5 124.5) (size 0.8) (drill 0.4) (layers F.Cu B.Cu) (net 69) (status 40000))
-  (via (at 121.5 122.5) (size 0.8) (drill 0.4) (layers F.Cu B.Cu) (net 69) (status 40000))
   (via (at 123.5 128.5) (size 0.8) (drill 0.4) (layers F.Cu B.Cu) (net 69) (status 40000))
   (via (at 123.5 126.5) (size 0.8) (drill 0.4) (layers F.Cu B.Cu) (net 69) (status 40000))
   (via (at 123.5 124.5) (size 0.8) (drill 0.4) (layers F.Cu B.Cu) (net 69) (status 40000))
-  (via (at 123.5 122.5) (size 0.8) (drill 0.4) (layers F.Cu B.Cu) (net 69) (status 40000))
   (via (at 125.5 128.5) (size 0.8) (drill 0.4) (layers F.Cu B.Cu) (net 69) (status 40000))
   (via (at 125.5 126.5) (size 0.8) (drill 0.4) (layers F.Cu B.Cu) (net 69) (status 40000))
   (via (at 125.5 124.5) (size 0.8) (drill 0.4) (layers F.Cu B.Cu) (net 69) (status 40000))
-  (via (at 125.5 122.5) (size 0.8) (drill 0.4) (layers F.Cu B.Cu) (net 69) (status 40000))
   (segment (start 77.25 95.75) (end 77.25 93) (width 2) (layer F.Cu) (net 69) (status 40000))
   (segment (start 94.25 95.75) (end 94.25 93) (width 2) (layer F.Cu) (net 69) (status 40000))
@@
   (segment (start 116.75 109) (end 116.75 96.5) (width 2) (layer F.Cu) (net 69) (status 40000))
   (segment (start 116.75 122.5) (end 116.75 109) (width 2) (layer F.Cu) (net 69) (status 40000))
-  (via (at 75.5 91.25) (size 0.8) (drill 0.4) (layers F.Cu B.Cu) (net 43) (status 40000))
-  (segment (start 75.5 94.75) (end 75.5 91.25) (width 0.25) (layer B.Cu) (net 43))
-  (segment (start 75.5 91.25) (end 76.5 91.25) (width 0.25) (layer F.Cu) (net 43))
-  (segment (start 76.5 91.25) (end 78.75 89) (width 0.25) (layer F.Cu) (net 43))
+  (segment (start 123.5 122.65) (end 123.5 116.25) (width 0.25) (layer F.Cu) (net 69))
   (segment (start 103.38 71.63) (end 103.38 73.63) (width 0.25) (layer F.Cu) (net 70))
   (segment (start 100.84 71.63) (end 100.84 73.34) (width 0.25) (layer F.Cu) (net 71))
@@
   (segment (start 93.22 86.87) (end 93.22 88.97) (width 0.25) (layer F.Cu) (net 84))
   (segment (start 90.68 86.87) (end 90.68 88.57) (width 0.25) (layer F.Cu) (net 85))
-  (zone (net 69) (net_name VCC2) (layer B.Cu) (hatch full 0.508)
-    (connect_pads thru_hole_only (clearance 0.5))
+  (zone (net 68) (net_name VCC1) (layer B.Cu) (hatch full 0.508)
+    (priority 1)
+    (connect_pads thru_hole_only (clearance 2))
     (min_thickness 0.2)
     (fill yes (arc_segments 32) (thermal_gap 0.5) (thermal_bridge_width 0.5) (smoothing fillet) (radius 0.5))
     (polygon
       (pts
-        (xy 130.751301 121.5) (xy 130.766142 136.5) (xy 115.758722 136.5) (xy 115.743881 121.5)
+        (xy 115.755098 36.9) (xy 115.740257 21.9) (xy 130.747677 21.9) (xy 130.762518 36.9)
       )
     )
   )
-  (zone (net 69) (net_name VCC2) (layer F.Cu) (hatch full 0.508)
-    (connect_pads thru_hole_only (clearance 0.5))
-    (min_thickness 0.2)
-    (fill yes (arc_segments 32) (thermal_gap 0.5) (thermal_bridge_width 0.5) (smoothing fillet) (radius 0.5))
+  (zone (net 1) (net_name GND) (layer B.Cu) (hatch edge 0.508)
+    (connect_pads (clearance 0.5))
+    (min_thickness 0.254)
+    (fill yes (arc_segments 32) (thermal_gap 0.508) (thermal_bridge_width 0.508))
     (polygon
       (pts
-        (xy 130.752286 121.5) (xy 130.767127 136.5) (xy 115.759707 136.5) (xy 115.744866 121.5)
+        (xy 152 138.5) (xy 44 138.5) (xy 44 20) (xy 152 20)
       )
     )
   )
   (zone (net 68) (net_name VCC1) (layer F.Cu) (hatch full 0.508)
-    (connect_pads thru_hole_only (clearance 0.5))
+    (priority 1)
+    (connect_pads thru_hole_only (clearance 2))
     (min_thickness 0.2)
     (fill yes (arc_segments 32) (thermal_gap 0.5) (thermal_bridge_width 0.5) (smoothing fillet) (radius 0.5))
     (polygon
       (pts
-        (xy 115.754358 36.897268) (xy 115.739517 21.897268) (xy 130.746937 21.897268) (xy 130.761778 36.897268)
+        (xy 115.755098 36.9) (xy 115.740257 21.9) (xy 130.747677 21.9) (xy 130.762518 36.9)
       )
     )
   )
-  (zone (net 68) (net_name VCC1) (layer B.Cu) (hatch full 0.508)
-    (connect_pads thru_hole_only (clearance 0.5))
+  (zone (net 69) (net_name VCC2) (layer F.Cu) (hatch full 0.508)
+    (priority 1)
+    (connect_pads thru_hole_only (clearance 2))
     (min_thickness 0.2)
     (fill yes (arc_segments 32) (thermal_gap 0.5) (thermal_bridge_width 0.5) (smoothing fillet) (radius 0.5))
     (polygon
       (pts
-        (xy 115.755098 36.9) (xy 115.740257 21.9) (xy 130.747677 21.9) (xy 130.762518 36.9)
+        (xy 130.756232 121.499988) (xy 130.771073 136.499988) (xy 115.763653 136.499988) (xy 115.748812 121.499988)
       )
     )
   )
-  (zone (net 0) (net_name "") (layer B.Cu) (hatch edge 0.508)
-    (connect_pads (clearance 0.5))
-    (min_thickness 0.254)
-    (fill yes (arc_segments 32) (thermal_gap 0.508) (thermal_bridge_width 0.508))
+  (zone (net 69) (net_name VCC2) (layer B.Cu) (hatch full 0.508)
+    (priority 1)
+    (connect_pads thru_hole_only (clearance 2))
+    (min_thickness 0.2)
+    (fill yes (arc_segments 32) (thermal_gap 0.5) (thermal_bridge_width 0.5) (smoothing fillet) (radius 0.5))
     (polygon
       (pts
-        (xy 152 138.5) (xy 44 138.5) (xy 44 20) (xy 152 20)
+        (xy 130.756232 121.499988) (xy 130.771073 136.499988) (xy 115.763653 136.499988) (xy 115.748812 121.499988)
       )
     )

Commit message: updates
Parts:
- moved C11 39.7 mm to (117.8, 83.8), turned to 90 degrees
- moved J9 21.0 mm to (129.0, 107.5), turned to 90 degrees
- moved C12 18.2 mm to (117.8, 71.2), turned to 270 degrees
- moved U11 14.5 mm to (127.0, 48.8)
Routing:
- net +5V: track 146.5 -> 128.5 mm
- net GND: track 112.6 -> 99.2 mm, vias 69 -> 67
- net +24V: track 31.1 -> 41.5 mm
Other:
- board outline added: 88.8 x 115.5 mm

Commit message: updates
Parts:
- R17, R18, R19, R20, R21, R22, R23, R24, R25, R26, R27, R28, R29, R30, R31, R32: footprint Resistor_SMD:R_0603_1608Metric_Pad1.05x0.95mm_HandSolder -> Resistor_SMD:R_1206_3216Metric_Pad1.42x1.75mm_HandSolder
- moved R31 6.26 mm to (92.5, 83.0), turned to 270 degrees
- moved R19 6.24 mm to (97.5, 75.5), turned to 270 degrees
- moved R22 6.20 mm to (89.9, 75.5), turned to 270 degrees
- moved R28 6.12 mm to (74.7, 83.0), turned to 90 degrees
- moved R29 6.01 mm to (79.8, 83.0), turned to 90 degrees
- moved R26 6.00 mm to (77.2, 75.5), turned to 270 degrees
- moved R32 6.00 mm to (89.9, 83.0), turned to 270 degrees
- moved R23 6.00 mm to (87.4, 75.5), turned to 270 degrees
- moved R25 6.00 mm to (82.3, 75.5), turned to 270 degrees
- moved R20 1.41 mm to (95.0, 75.5)
- moved R18 1.35 mm to (100.1, 75.5)
- moved R24 1.35 mm to (84.8, 75.5)
- moved R17 1.33 mm to (102.6, 75.5)
- moved R27 1.31 mm to (72.2, 75.5)
- moved R21 1.27 mm to (92.5, 75.5)
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Connections:
- R21 pad 2: R_2 -> R_7
- R26 pad 2: R_4 -> R_5
- R27 pad 2: R_5 -> R_4
- R30 pad 2: R_7 -> R_2
Routing:
- net R_3: track 49.3 -> 14.3 mm
- net T_1: track 22.6 -> 33.4 mm
- net T_7: track 18.8 -> 26.4 mm
- net T_5: track 36.6 -> 43.9 mm
- net T_2: track 17.6 -> 24.8 mm
- net R_2: track 29.2 -> 36.0 mm
- net T_8: track 22.3 -> 28.9 mm
- net T_4: track 40.3 -> 46.8 mm
- net T_3: track 28.6 -> 34.8 mm
- net R_6: track 18.4 -> 24.3 mm
- net R_5: track 48.2 -> 44.5 mm
- net R_1: track 27.0 -> 25.1 mm
- net R_4: track 42.1 -> 43.2 mm
- net Net-(R30-Pad1): track 1.81 -> 2.81 mm
- net Net-(R19-Pad1): track 1.83 -> 2.82 mm
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
Commit message: wip
Parts:
- R17, R18, R19, R20, R21, R22, R23, R24, R25, R26, R27, R28, R29, R30, R31, R32: footprint Resistor_SMD:R_1206_3216Metric_Pad1.42x1.75mm_HandSolder -> Resistor_SMD:R_0805_2012Metric_Pad1.15x1.40mm_HandSolder
- moved C1 1.58 mm to (98.5, 46.4)
- moved C2 1.58 mm to (81.5, 46.4)
- moved C3 1.58 mm to (64.5, 46.4)
- moved C4 1.58 mm to (47.5, 46.4)
- moved C5 1.58 mm to (60.2, 112.1)
- moved C6 1.58 mm to (77.2, 112.1)
- moved C7 1.58 mm to (94.2, 112.1)
- moved C8 1.58 mm to (111.2, 112.1)
- moved R1 1.58 mm to (107.5, 42.8)
- moved R10 1.58 mm to (57.2, 115.8)
- moved R11 1.58 mm to (68.2, 115.8)
- moved R12 1.58 mm to (74.2, 115.8)
- moved R13 1.58 mm to (85.2, 115.8)
- moved R14 1.58 mm to (91.2, 115.8)
- moved R15 1.58 mm to (102.2, 115.8)
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Connections:
- R18 pad 2: R_1 -> R_7
- R20 pad 2: R_3 -> R_1
- R21 pad 2: R_7 -> R_2
- R26 pad 2: R_5 -> R_3
- R29 pad 2: R_6 -> R_5
- R30 pad 2: R_2 -> R_6
Routing:
- net VCC1: track 232.2 -> 211.8 mm, vias 30 -> 22
- net R_3: track 14.3 -> 31.9 mm
- net R_7: track 29.6 -> 36.2 mm
- net R_6: track 24.3 -> 30.3 mm
- net R_2: track 36.0 -> 32.3 mm
- net VCC2: track 211.7 -> 208.9 mm, vias 30 -> 22
- net Net-(J7-Pad1): track 13.8 -> 11.0 mm
- net T_1: track 33.4 -> 30.9 mm
- net Net-(J8-Pad7): track 13.8 -> 11.7 mm
- net Net-(J7-Pad7): track 13.8 -> 11.7 mm
- net Net-(J6-Pad7): track 13.8 -> 11.7 mm
- net Net-(J5-Pad7): track 13.8 -> 11.7 mm
- net Net-(J4-Pad7): track 13.8 -> 11.7 mm
- net Net-(J3-Pad7): track 13.8 -> 11.7 mm
- net Net-(J2-Pad7): track 13.8 -> 11.7 mm
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Other:
- board size 88.8 x 115.5 mm -> 89.2 x 115.5 mm

Commit message: wip
Parts:
- moved J9 115.4 mm to (48.0, 25.3), turned to 270 degrees
- moved U11 84.8 mm to (49.9, 84.0), turned to 180 degrees
- moved C11 75.2 mm to (59.8, 35.9), turned to 0 degrees
- moved U10 68.7 mm to (57.5, 100.5)
- moved C12 68.1 mm to (51.6, 87.4), turned to 0 degrees
- moved U9 67.4 mm to (57.8, 54.9), turned to 270 degrees
- moved C10 55.9 mm to (61.1, 90.4)
- moved C9 51.5 mm to (63.6, 53.2), turned to 90 degrees
- moved RX_SW1 32.6 mm to (131.2, 44.8), turned to 90 degrees
- moved RX_SW2 32.6 mm to (114.2, 44.8), turned to 90 degrees
- moved RX_SW3 32.6 mm to (97.2, 44.8), turned to 90 degrees
- moved RX_SW4 32.6 mm to (80.2, 44.8), turned to 90 degrees
- moved J5 29.4 mm to (68.8, 100.5)
- moved J6 29.4 mm to (85.8, 100.5)
- moved J7 29.4 mm to (102.8, 100.5)
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Connections:
- J9 pad 1: +24V -> GND
- J9 pad 2: GND -> +24V
Routing:
- net GND: track 99.2 -> 159.8 mm, vias 67 -> 52
- net +5V: track 128.5 -> 163.6 mm
- net VCC1: track 211.8 -> 179.3 mm
- net VCC2: track 208.9 -> 190.2 mm
- net +24V: track 41.5 -> 24.2 mm
- net R_2: track 32.3 -> 21.0 mm
- net T_5: track 44.4 -> 33.5 mm
- net T_1: track 30.9 -> 20.2 mm
- net R_4: track 42.4 -> 31.6 mm
- net R_3: track 31.9 -> 21.2 mm
- net T_7: track 26.4 -> 15.9 mm
- net R_8: track 35.2 -> 25.0 mm, vias 2 -> 4
- net R_5: track 44.0 -> 34.9 mm
- net T_6: track 40.6 -> 32.2 mm, vias 2 -> 4
- net T_8: track 30.7 -> 22.7 mm
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Other:
- board size 89.2 x 115.5 mm -> 91.2 x 93.5 mm

Commit message: wip
Parts:
- C1: renamed from C4; footprint Capacitor_SMD:C_0603_1608Metric_Pad1.05x0.95mm_HandSolder -> Capacitor_SMD:C_0603_1608Metric
- C10, C12, C9: footprint Capacitor_Tantalum_SMD:CP_EIA-3528-21_Kemet-B_Pad1.50x2.35mm_HandSolder -> Capacitor_Tantalum_SMD:CP_EIA-3528-21_Kemet-B
- C2: renamed from C3; footprint Capacitor_SMD:C_0603_1608Metric_Pad1.05x0.95mm_HandSolder -> Capacitor_SMD:C_0603_1608Metric
- C3: renamed from C2; footprint Capacitor_SMD:C_0603_1608Metric_Pad1.05x0.95mm_HandSolder -> Capacitor_SMD:C_0603_1608Metric
- C4: renamed from C1; footprint Capacitor_SMD:C_0603_1608Metric_Pad1.05x0.95mm_HandSolder -> Capacitor_SMD:C_0603_1608Metric
- C5: renamed from C8; footprint Capacitor_SMD:C_0603_1608Metric_Pad1.05x0.95mm_HandSolder -> Capacitor_SMD:C_0603_1608Metric
- C6: renamed from C7; footprint Capacitor_SMD:C_0603_1608Metric_Pad1.05x0.95mm_HandSolder -> Capacitor_SMD:C_0603_1608Metric
- C7: renamed from C6; footprint Capacitor_SMD:C_0603_1608Metric_Pad1.05x0.95mm_HandSolder -> Capacitor_SMD:C_0603_1608Metric
- C8: renamed from C5; footprint Capacitor_SMD:C_0603_1608Metric_Pad1.05x0.95mm_HandSolder -> Capacitor_SMD:C_0603_1608Metric
- R1: renamed from R7; footprint Resistor_SMD:R_1206_3216Metric_Pad1.42x1.75mm_HandSolder -> Resistor_SMD:R_1206_3216Metric
- R10: renamed from R16; footprint Resistor_SMD:R_1206_3216Metric_Pad1.42x1.75mm_HandSolder -> Resistor_SMD:R_1206_3216Metric
- R11: renamed from R13; footprint Resistor_SMD:R_1206_3216Metric_Pad1.42x1.75mm_HandSolder -> Resistor_SMD:R_1206_3216Metric
- R12: renamed from R14; footprint Resistor_SMD:R_1206_3216Metric_Pad1.42x1.75mm_HandSolder -> Resistor_SMD:R_1206_3216Metric
- R13: renamed from R11; footprint Resistor_SMD:R_1206_3216Metric_Pad1.42x1.75mm_HandSolder -> Resistor_SMD:R_1206_3216Metric
- R14: renamed from R12; footprint Resistor_SMD:R_1206_3216Metric_Pad1.42x1.75mm_HandSolder -> Resistor_SMD:R_1206_3216Metric
- R15: renamed from R9; footprint Resistor_SMD:R_1206_3216Metric_Pad1.42x1.75mm_HandSolder -> Resistor_SMD:R_1206_3216Metric
- R16: renamed from R10; footprint Resistor_SMD:R_1206_3216Metric_Pad1.42x1.75mm_HandSolder -> Resistor_SMD:R_1206_3216Metric
- R17, R18, R19, R20, R21, R22, R23, R24, R25, R26, R27, R28, R29, R30, R31, R32: footprint Resistor_SMD:R_0805_2012Metric_Pad1.15x1.40mm_HandSolder -> Resistor_SMD:R_0805_2012Metric
- R2: renamed from R8; footprint Resistor_SMD:R_1206_3216Metric_Pad1.42x1.75mm_HandSolder -> Resistor_SMD:R_1206_3216Metric
- R3: renamed from R5; footprint Resistor_SMD:R_1206_3216Metric_Pad1.42x1.75mm_HandSolder -> Resistor_SMD:R_1206_3216Metric
- R4: renamed from R6; footprint Resistor_SMD:R_1206_3216Metric_Pad1.42x1.75mm_HandSolder -> Resistor_SMD:R_1206_3216Metric
- R5: renamed from R3; footprint Resistor_SMD:R_1206_3216Metric_Pad1.42x1.75mm_HandSolder -> Resistor_SMD:R_1206_3216Metric
- R6: renamed from R4; footprint Resistor_SMD:R_1206_3216Metric_Pad1.42x1.75mm_HandSolder -> Resistor_SMD:R_1206_3216Metric
- R7: renamed from R1; footprint Resistor_SMD:R_1206_3216Metric_Pad1.42x1.75mm_HandSolder -> Resistor_SMD:R_1206_3216Metric
- R8: renamed from R2; footprint Resistor_SMD:R_1206_3216Metric_Pad1.42x1.75mm_HandSolder -> Resistor_SMD:R_1206_3216Metric
- R9: renamed from R15; footprint Resistor_SMD:R_1206_3216Metric_Pad1.42x1.75mm_HandSolder -> Resistor_SMD:R_1206_3216Metric
- moved C11 32.4 mm to (59.0, 68.2), turned to 270 degrees
- moved U9 18.9 mm to (57.0, 36.0), turned to 90 degrees
- moved J9 12.2 mm to (48.0, 37.5)
- moved C10 10.9 mm to (64.2, 80.0), turned to 90 degrees
- moved U11 10.0 mm to (49.9, 94.0)
- moved C12 5.02 mm to (56.2, 85.5), turned to 90 degrees
- moved C9 3.55 mm to (63.8, 56.8), turned to 270 degrees
- moved U10 0.50 mm to (57.0, 100.5)
- renumbered TX_SW4 to DE1, TX_SW3 to DE2, TX_SW2 to DE3, TX_SW1 to DE4, TX_SW8 to DE5, TX_SW7 to DE6, TX_SW6 to DE7, TX_SW5 to DE8, J4 to J1, J3 to J2, J2 to J3, J1 to J4, J8 to J5, J7 to J6, J6 to J7, J5 to J8, RX_SW4 to RE1, RX_SW3 to RE2, RX_SW2 to RE3, RX_SW1 to RE4, RX_SW8 to RE5, RX_SW7 to RE6, RX_SW6 to RE7, RX_SW5 to RE8, U4 to U1, U3 to U2, U2 to U3, U1 to U4, U8 to U5, U7 to U6, U6 to U7, U5 to U8
Routing:
- net +5V: track 163.6 -> 149.1 mm
- net +24V: track 24.2 -> 37.4 mm
- net VCC1: track 179.3 -> 189.0 mm
- net Net-(J8-Pad8): track 9.82 -> 8.85 mm
- net Net-(J7-Pad8): track 9.82 -> 8.85 mm
- net Net-(J6-Pad8): track 9.82 -> 8.85 mm
- net GND: track 159.8 -> 158.9 mm, vias 52 -> 56
- net Net-(J8-Pad1): track 11.5 -> 10.7 mm
- net Net-(J7-Pad1): track 11.5 -> 10.7 mm
- net Net-(J6-Pad1): track 11.5 -> 10.7 mm
- net Net-(J1-Pad1): track 18.2 -> 17.4 mm
- net R_7: track 28.3 -> 28.8 mm
Other:
- outline, holes or cut-outs redrawn
