File: TheListener/Mothership/Mothership.kicad_pcb (KiCad board)
At the start: 2 copper layers, 91.2 x 93.5 mm, 81 parts, among them J1 RJ45, J2 RJ45, J3 RJ45, J4 RJ45, J5 RJ45, J6 RJ45, J7 RJ45, J8 RJ45, J9 Conn_01x02_Female, U1 SP3491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

Commit message: updates and plots
Parts:
- added REF**: MountingHole_3.2mm_M3, MountingHole:MountingHole_3.2mm_M3, F.Cu at (49.8, 39.0)
- added REF**: MountingHole_3.2mm_M3, MountingHole:MountingHole_3.2mm_M3, F.Cu at (43.0, 99.0)
- added REF**: MountingHole_3.2mm_M3, MountingHole:MountingHole_3.2mm_M3, F.Cu at (136.2, 30.0)
- added REF**: MountingHole_3.2mm_M3, MountingHole:MountingHole_3.2mm_M3, F.Cu at (136.2, 106.5)
- added REF**: JLCPCB SMT Tooling Hole, TheListener:JLCPCB SMT Tooling Hole, F.Cu at (40.2, 112.5)
- added REF**: JLCPCB SMT Tooling Hole, TheListener:JLCPCB SMT Tooling Hole, F.Cu at (137.2, 24.0)
- added REF**: JLCPCB SMT Tooling Hole, TheListener:JLCPCB SMT Tooling Hole, F.Cu at (137.2, 112.5)
- moved J9 5.20 mm to (42.8, 37.5)
Routing:
- net +24V: track 37.4 -> 33.6 mm
- net GND: track 158.9 -> 160.2 mm
Other:
- board size 91.2 x 93.5 mm -> 102 x 93.5 mm

Commit message: updated plots and drills
Parts:
- moved REF** 9.00 mm to (136.2, 39.0)
- moved REF** 7.50 mm to (136.2, 99.0)
- moved REF** 6.75 mm to (49.8, 99.0)
Changed lines of the file:
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@@
   )
   (module MountingHole:MountingHole_3.2mm_M3 (layer F.Cu)
-    (at 43 99)
+    (at 49.75 99)
     (descr "Mounting Hole 3.2mm, no annular, M3")
     (tags "mounting hole 3.2mm no annular m3")
@@
   )
   (module MountingHole:MountingHole_3.2mm_M3 (layer F.Cu)
-    (at 136.25 30 180)
+    (at 136.25 39 180)
     (descr "Mounting Hole 3.2mm, no annular, M3")
     (tags "mounting hole 3.2mm no annular m3")
@@
   )
   (module MountingHole:MountingHole_3.2mm_M3 (layer F.Cu)
-    (at 136.25 106.5)
+    (at 136.25 99)
     (descr "Mounting Hole 3.2mm, no annular, M3")
     (tags "mounting hole 3.2mm no annular m3")

Commit message: receiver, updates, desk bom
Parts:
- removed REF** (x4): MountingHole_3.2mm_M3, MountingHole:MountingHole_3.2mm_M3
- removed REF** (x3): JLCPCB SMT Tooling Hole, TheListener:JLCPCB SMT Tooling Hole
- moved C10 0.50 mm to (63.8, 80.0)
Routing:
- net GND: track 160.2 -> 131.8 mm
- net T_8: track 22.7 -> 22.0 mm
- net VCC1: track 189.0 -> 189.7 mm
- net +24V: track 33.6 -> 34.1 mm

Commit message: wip
Parts:
- removed J9: Conn_01x02_Female, TerminalBlock_Phoenix:TerminalBlock_Phoenix_PT-1,5-2-3.5-H_1x02_P3.50mm_Horizontal
- removed R17, R18, R19, R20, R21, R22, R23, R24, R25, R26, R27, R28, R29, R30, R31, R32: 220, Resistor_SMD:R_0805_2012Metric
- removed U11: NID35-5, TheListener:Converter_DCDC_MeanWell_NID35_THT
- removed U12: Teensy3.5, TheListener:Teensy35_36_NoMiddlePins
- added J10: Conn_01x10_Female, Connector_PinHeader_2.54mm:PinHeader_1x10_P2.54mm_Vertical, F.Cu at (85.8, 61.2)
- added J11: Conn_01x10_Female, Connector_PinHeader_2.54mm:PinHeader_1x10_P2.54mm_Vertical, F.Cu at (108.5, 74.5)
- C11: value 100uF -> 22uF; footprint Capacitor_SMD:CP_Elec_8x10 -> Capacitor_Tantalum_SMD:CP_EIA-3528-21_Kemet-B
- moved U9 63.6 mm to (112.0, 68.0), turned to 0 degrees
- moved C9 49.5 mm to (113.0, 61.2), turned to 180 degrees
- moved C11 46.8 mm to (105.8, 68.0), turned to 90 degrees
- moved U10 41.0 mm to (82.0, 68.0), turned to 180 degrees
- moved C12 36.5 mm to (88.2, 68.0), turned to 270 degrees
- moved C10 18.3 mm to (81.2, 74.8), turned to 0 degrees
- moved C1 0.25 mm to (67.2, 45.4)
- moved C2 0.25 mm to (84.2, 45.4)
- moved C3 0.25 mm to (101.2, 45.4)
- moved C4 0.25 mm to (118.2, 45.4)
- moved DE1 0.25 mm to (80.0, 51.2)
- moved DE2 0.25 mm to (97.0, 51.2)
- moved DE3 0.25 mm to (114.0, 51.2)
- moved DE4 0.25 mm to (131.0, 51.2)
- moved J1 0.25 mm to (77.8, 36.0)
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Connections:
- C1 pad 2: VCC1 -> VCC2
- C11 pad 1: +24V -> +5V
- C2 pad 2: VCC1 -> VCC2
- C5 pad 2: VCC2 -> VCC1
- C6 pad 2: VCC2 -> VCC1
- DE1 pad 1: VCC1 -> VCC2
- DE2 pad 1: VCC1 -> VCC2
- DE5 pad 1: VCC2 -> VCC1
- DE6 pad 1: VCC2 -> VCC1
- RE1 pad 3: VCC1 -> VCC2
- RE2 pad 3: VCC1 -> VCC2
- RE5 pad 3: VCC2 -> VCC1
- RE6 pad 3: VCC2 -> VCC1
- U1 pad 14: VCC1 -> VCC2
- U2 pad 14: VCC1 -> VCC2
- U5 pad 14: VCC2 -> VCC1
- U6 pad 14: VCC2 -> VCC1
Routing:
- net +5V: track 149.1 -> 34.5 mm
- net +24V: track 34.1 -> 0.00 mm
- net GND: track 131.8 -> 110.7 mm, vias 56 -> 92
- net T_6: track 32.2 -> 12.1 mm, vias 4 -> 2
- net VCC1: track 189.7 -> 205.7 mm, vias 22 -> 0
- net T_4: track 39.7 -> 24.2 mm
- net T_3: track 27.6 -> 12.3 mm
- net R_5: track 34.9 -> 22.0 mm
- net R_6: track 23.3 -> 11.5 mm
- net R_7: track 28.8 -> 17.1 mm, vias 4 -> 2
- net T_5: track 33.5 -> 23.3 mm
- net VCC2: track 190.2 -> 199.4 mm, vias 22 -> 0
- net R_2: track 21.0 -> 13.1 mm
- net R_3: track 21.2 -> 13.5 mm
- net T_1: track 20.2 -> 26.9 mm
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- removed copper zone on B.Cu, net VCC1
- removed copper zone on F.Cu, net VCC1
- removed copper zone on B.Cu, net VCC2
- removed copper zone on F.Cu, net VCC2
Other:
- board size 102 x 93.5 mm -> 82 x 93.5 mm

Commit message: updates
Parts:
- added C13: 10uF, Capacitor_Tantalum_SMD:CP_EIA-3528-21_Kemet-B, F.Cu at (120.5, 73.8)
- added C14: 10uF, Capacitor_Tantalum_SMD:CP_EIA-3528-21_Kemet-B, F.Cu at (77.8, 62.5)
- C10, C9: value 22uF -> 10uF
- J10, J11: value Conn_01x10_Female -> Conn_02x05_Odd_Even; footprint Connector_PinHeader_2.54mm:PinHeader_1x10_P2.54mm_Vertical -> Connector_PinSocket_2.54mm:PinSocket_2x05_P2.54mm_Vertical
- moved J10 12.1 mm to (87.2, 73.2), turned to 180 degrees
- moved J11 11.8 mm to (111.0, 63.0), turned to 0 degrees
- moved C11 9.00 mm to (114.8, 67.8)
- moved U9 9.00 mm to (121.0, 68.2)
- moved C9 7.65 mm to (120.5, 62.8)
- moved C12 4.76 mm to (83.5, 68.2)
- moved U10 4.75 mm to (77.2, 68.0)
- moved C10 3.72 mm to (77.8, 73.5)
Connections:
- J10 pad 1: +5V -> T_5
- J10 pad 10: GND -> R_3
- J10 pad 2: R_4 -> R_5
- J10 pad 3: T_4 -> GND
- J10 pad 4: R_3 -> T_6
- J10 pad 5: T_3 -> +5V
- J10 pad 6: R_2 -> R_6
- J10 pad 7: T_2 -> R_4
- J10 pad 8: R_1 -> T_3
- J10 pad 9: T_1 -> T_4
- J11 pad 1: +5V -> T_1
- J11 pad 10: GND -> R_7
- J11 pad 2: R_8 -> R_1
- J11 pad 3: T_8 -> GND
- J11 pad 4: R_7 -> T_2
- J11 pad 5: T_7 -> +5V
- J11 pad 6: R_6 -> R_2
- J11 pad 7: T_6 -> R_8
- J11 pad 8: R_5 -> T_7
- J11 pad 9: T_5 -> T_8
Routing:
- net +5V: track 34.5 -> 15.7 mm
- net VCC1: track 205.7 -> 193.6 mm
- net GND: track 110.7 -> 118.9 mm, vias 92 -> 100
- net R_6: track 11.5 -> 18.8 mm
- net T_8: track 27.8 -> 20.7 mm
- net R_2: track 13.1 -> 18.6 mm
- net T_1: track 26.9 -> 21.5 mm
- net R_7: track 17.1 -> 12.9 mm
- net R_1: track 25.1 -> 20.9 mm
- net T_6: track 12.1 -> 16.0 mm
- net T_4: track 24.2 -> 21.3 mm
- net VCC2: track 199.4 -> 196.8 mm
- net R_8: track 28.8 -> 26.4 mm
- net T_3: track 12.3 -> 14.7 mm
- net T_2: track 14.4 -> 15.8 mm
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
Commit message: final
Parts:
- removed R1, R11, R13, R15, R3, R5, R7, R9: 100, Resistor_SMD:R_1206_3216Metric
- moved J1 3.25 mm to (77.8, 39.2)
- moved J2 3.25 mm to (94.8, 39.2)
- moved J3 3.25 mm to (111.8, 39.2)
- moved J4 3.25 mm to (128.8, 39.2)
- moved R2 3.25 mm to (70.8, 46.0)
- moved R4 3.25 mm to (87.8, 46.0)
- moved R6 3.25 mm to (104.8, 46.0)
- moved R8 3.25 mm to (121.8, 46.0)
- moved J5 2.75 mm to (119.8, 97.8)
- moved J6 2.75 mm to (102.8, 97.8)
- moved J7 2.75 mm to (85.8, 97.8)
- moved J8 2.75 mm to (68.8, 97.8)
- moved R10 2.75 mm to (126.7, 91.0)
- moved R12 2.75 mm to (109.7, 91.0)
- moved R14 2.75 mm to (92.7, 91.0)
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Connections:
- C11 pad 1: +5V -> 5VDC_1
- C12 pad 1: +5V -> 5VDC_2
- J10 pad 5: +5V -> 5VDC_2
- J11 pad 5: +5V -> 5VDC_1
- U10 pad 3: +5V -> 5VDC_2
- U9 pad 3: +5V -> 5VDC_1
Routing:
- net +5V: track 15.7 -> 0.00 mm
- net VCC2: track 196.8 -> 207.2 mm, vias 0 -> 22
- net GND: track 118.9 -> 108.7 mm, vias 100 -> 48
- net VCC1: track 193.6 -> 203.1 mm, vias 0 -> 22
- net 5VDC_1: track 0.00 -> 8.83 mm
- net 5VDC_2: track 0.00 -> 7.87 mm
- net Net-(J1-Pad1): track 17.4 -> 11.3 mm
- net T_7: track 15.5 -> 12.9 mm
- net T_5: track 23.7 -> 21.6 mm
- net T_6: track 16.0 -> 13.9 mm
- net R_3: track 12.7 -> 10.6 mm
- net R_7: track 12.9 -> 10.9 mm
- net T_2: track 15.8 -> 14.3 mm
- net R_6: track 18.8 -> 17.4 mm
- net T_3: track 14.7 -> 13.3 mm
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- added copper zone on B.Cu, net VCC1
- added copper zone on F.Cu, net VCC1
- added copper zone on B.Cu, net VCC2
- added copper zone on F.Cu, net VCC2
Other:
- board size 82 x 93.5 mm -> 82.2 x 87.5 mm

Commit message: working
Parts:
- added J12: Conn_01x04_Male, Connector_PinSocket_2.54mm:PinSocket_1x04_P2.54mm_Vertical, F.Cu at (111.8, 63.5)
- added J9: Conn_01x04_Male, Connector_PinSocket_2.54mm:PinSocket_1x04_P2.54mm_Vertical, F.Cu at (86.4, 73.6)
- moved J10 4.56 mm to (91.4, 73.6)
- moved J11 3.05 mm to (106.7, 63.5)
- moved C1 0.62 mm to (67.9, 47.9)
- moved C10 0.62 mm to (77.6, 74.0)
- moved C14 0.62 mm to (77.6, 63.2)
- moved C2 0.62 mm to (84.9, 47.9)
- moved C7 0.62 mm to (96.9, 89.1)
- moved C8 0.62 mm to (79.9, 89.1)
- moved DE1 0.62 mm to (80.6, 53.8)
- moved DE2 0.62 mm to (97.6, 53.8)
- moved DE7 0.62 mm to (84.1, 83.2)
- moved DE8 0.62 mm to (67.1, 83.2)
- moved J1 0.62 mm to (78.4, 39.2)
- moved J2 0.62 mm to (95.4, 39.2)
- moved J7 0.62 mm to (86.4, 97.8)
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Connections:
- J10 pad 1: T_5 -> R_5
- J10 pad 2: R_5 -> T_6
- J10 pad 3: GND -> T_5
- J10 pad 4: T_6 -> R_6
- J10 pad 5: 5VDC_2 -> (no net)
- J10 pad 6: R_6 -> (no net)
- J11 pad 1: T_1 -> R_1
- J11 pad 2: R_1 -> T_2
- J11 pad 3: GND -> T_1
- J11 pad 4: T_2 -> R_2
- J11 pad 5: 5VDC_1 -> (no net)
- J11 pad 6: R_2 -> (no net)
Routing:
- net T_5: track 21.6 -> 28.0 mm
- net T_1: track 22.6 -> 28.0 mm
- net VCC1: track 203.1 -> 207.2 mm, vias 22 -> 19
- net T_4: track 20.2 -> 24.1 mm
- net R_6: track 17.4 -> 14.0 mm
- net R_2: track 17.3 -> 14.0 mm
- net R_4: track 25.6 -> 28.9 mm
- net T_7: track 12.9 -> 16.0 mm
- net R_8: track 25.8 -> 28.9 mm
- net T_8: track 21.0 -> 24.1 mm
- net T_2: track 14.3 -> 11.4 mm
- net R_3: track 10.6 -> 13.4 mm
- net GND: track 108.7 -> 106.0 mm
- net T_3: track 13.3 -> 16.0 mm
- net T_6: track 13.9 -> 11.4 mm
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
Commit message: wip
Parts:
- removed J12, J9: Conn_01x04_Male, Connector_PinSocket_2.54mm:PinSocket_1x04_P2.54mm_Vertical
Connections:
- J10 pad 5: (no net) -> 5VDC_2
- J10 pad 6: (no net) -> GND
- J11 pad 5: (no net) -> 5VDC_1
- J11 pad 6: (no net) -> GND
Routing:
- net GND: track 106.0 -> 108.8 mm, vias 48 -> 52
- net 5VDC_2: track 9.65 -> 12.2 mm
- net 5VDC_1: track 9.65 -> 12.2 mm
